File: RICM Greenpower Telemetry Module/RICM Greenpower Instrument Cluster/RICM Greenpower Instrument Cluster.kicad_pcb (KiCad board)
At the start: 2 copper layers, 110 x 43.2 mm, 11 parts, among them J1 Conn_02x04_Counter_Clockwise

Commit message: update cluster
Updated cluster schematic to use an I2C gpio expander. Added two pushbutton switches.
Parts:
- added R5: R, Resistor_THT:R_Axial_DIN0207_L6.3mm_D2.5mm_P7.62mm_Horizontal, F.Cu at (43.2, 33.0)
- added R6: R, Resistor_THT:R_Axial_DIN0207_L6.3mm_D2.5mm_P7.62mm_Horizontal, F.Cu at (43.2, 29.2)
- added SW1: SW_Push, Button_Switch_THT:SW_PUSH_6mm_2pin, F.Cu at (10.7, 28.2)
- added SW2: SW_Push, Button_Switch_THT:SW_PUSH_6mm_2pin, F.Cu at (78.0, 28.2)
- added U1: PCA9555D, Package_SO:SOIC-24W_7.5x15.4mm_P1.27mm, B.Cu at (81.3, 14.7)
- J1: footprint Connector_PinHeader_2.54mm:PinHeader_2x04_P2.54mm_Vertical -> Connector_PinHeader_2.54mm:PinHeader_1x04_P2.54mm_Vertical
- moved DS1 1.27 mm to (81.3, 26.6)
- moved DS2 1.27 mm to (14.0, 26.6)
Connections:
- R1 pad 1: Net-(J1-Pad8) -> Net-(R1-Pad1)
- R2 pad 1: Net-(J1-Pad7) -> Net-(R2-Pad1)
- R3 pad 1: Net-(J1-Pad6) -> Net-(R3-Pad1)
- R4 pad 1: Net-(J1-Pad5) -> Net-(R4-Pad1)
Routing:
- net Net-(R5-Pad1): track 0.00 -> 86.2 mm
- net GND: track 102.4 -> 185.2 mm, vias 0 -> 1
- net Net-(R4-Pad1): track 0.00 -> 72.6 mm, vias 0 -> 2
- net Net-(R3-Pad1): track 0.00 -> 67.3 mm, vias 0 -> 2
- net Net-(R6-Pad1): track 0.00 -> 56.6 mm
- net Net-(R2-Pad1): track 0.00 -> 35.2 mm, vias 0 -> 2
- net Net-(R1-Pad1): track 0.00 -> 25.4 mm, vias 0 -> 2
- net Net-(J1-Pad5): track 24.5 -> 0.00 mm, vias 1 -> 0
- net +5V: track 99.9 -> 120.3 mm, vias 0 -> 1
- net SCL: track 92.5 -> 112.6 mm, vias 2 -> 3
- net Net-(J1-Pad6): track 15.0 -> 0.00 mm, vias 1 -> 0
- net SDA: track 100.3 -> 113.9 mm, vias 2 -> 3
- net Net-(J1-Pad8): track 12.5 -> 0.00 mm
- net Net-(J1-Pad7): track 7.84 -> 0.00 mm

Commit message: last revisions before first order
Parts:
- moved J1 22.4 mm to (22.9, 32.8)
- moved D4 22.4 mm to (12.7, 19.3)
- moved DS1 22.4 mm to (61.0, 36.1)
- moved DS2 22.4 mm to (-6.31, 36.1)
- moved R1 22.4 mm to (42.2, 32.3)
- moved R2 22.4 mm to (38.1, 32.3)
- moved SW1 22.4 mm to (-9.56, 37.7)
- moved SW2 22.4 mm to (57.8, 37.7)
- moved U1 22.4 mm to (61.0, 24.2)
- moved D2 22.4 mm to (30.5, 19.6)
- moved D3 22.4 mm to (21.6, 19.3)
- moved R3 22.4 mm to (16.6, 32.1)
- moved R4 22.4 mm to (12.5, 32.1)
- moved R5 22.4 mm to (22.9, 42.5)
- moved R6 22.4 mm to (22.9, 38.7)
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
Commit message: Similar corrections for display module
Fixed pinout and updated silkscreen and notes for the display module schematic and board.
Connections:
- DS1 pad 2: +5V -> +3V3
- DS2 pad 2: +5V -> +3V3
- J1 pad 1: +5V -> GND
- J1 pad 2: GND -> +3V3
- J1 pad 3: SDA -> SCL
- J1 pad 4: SCL -> SDA
- U1 pad 24: +5V -> +3V3
Routing:
- net +5V: track 120.3 -> 12.7 mm, vias 1 -> 0
- net +3V3: track 0.00 -> 105.1 mm, vias 0 -> 1
- net SCL: track 112.6 -> 107.1 mm
- net SDA: track 113.9 -> 114.8 mm
- net GND: track 185.2 -> 184.6 mm
