File: RICM Greenpower Telemetry Module/RICM Greenpower Instrument Cluster/RICM Greenpower Instrument Cluster.kicad_sch (KiCad schematic)
At the start: 16 parts, among them J1 Conn_02x04_Counter_Clockwise, SW1 SW_Push, SW2 SW_Push, U1 PCA9555D

Commit message: Similar corrections for display module
Fixed pinout and updated silkscreen and notes for the display module schematic and board.
Connections:
- net GND: now also J1.1 (Pin_1); no longer J1.2 (Pin_2)
- net SCL: now also J1.3 (Pin_3); no longer J1.4 (Pin_4)
- net SDA: now also J1.4 (Pin_4); no longer J1.3 (Pin_3)
- net +5V renamed +3V3
- net +3V3: now also J1.2 (Pin_2); no longer J1.1 (Pin_1)
Other:
- note added: "N.B.! DO NOT FORGET to switch the address jumper on one screen before installing them"
